File: hardware/jst-zh/adafruit-3309-adapter-zh.kicad_pcb (KiCad board)
At the start: 2 copper layers, 20.3 x 33 mm, 3 parts, among them J1 S6B-ZR-SM4A-TF(LF)(SN), J2 Conn_01x08_Female, J3 Conn_01x08_Female

Commit message: Routing done
Routing:
- net /DTR: track 0.00 -> 23.0 mm
- net /RTS: track 0.00 -> 19.6 mm
- net /TX: track 0.00 -> 17.3 mm
- net /RX: track 0.00 -> 11.1 mm
- net GND: track 0.00 -> 6.08 mm, vias 0 -> 4
- added copper zone on F.Cu, net +5V
- added copper zone on B.Cu, net GND

Commit message: Add version of previous commit
Other:
- board text added: "François Gervais 31 jan 2021 v1.0.0"
Changed lines of the file:
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@@
   (general
     (thickness 1.6)
-    (drawings 11)
+    (drawings 12)
     (tracks 26)
     (zones 0)
@@
     )
   )
+  (gr_text "François Gervais\n31 jan 2021\nv1.0.0" (at 53.675001 27.125001) (layer B.SilkS)
+    (effects (font (size 1 1) (thickness 0.15)) (justify left mirror))
+  )
   (gr_arc (start 54.931001 55.921001) (end 54.931001 56.175001) (angle -90) (layer Edge.Cuts) (width 0.05))
