File: hardware/jst-sh/adafruit-3309-adapter.kicad_pcb (KiCad board)
At the start: 2 copper layers, 20.3 x 33 mm, 3 parts, among them J1 SM06B-SRSS-TB(LF)(SN), J2 Conn_01x08_Female, J3 Conn_01x08_Female

Commit message: Add version of previous commit
Other:
- board text added: "François Gervais 2 fev 2021 v1.0.0-2-g5c36f27"
- board text removed: "François Gervais 2 fev 2021 v"
Changed lines of the file:
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@@
     )
   )
-  (gr_text "François Gervais\n2 fev 2021\nv" (at 53.675001 27.125001) (layer B.SilkS)
+  (gr_text "François Gervais\n2 fev 2021\nv1.0.0-2-g5c36f27" (at 53.675001 27.125001) (layer B.SilkS)
     (effects (font (size 1 1) (thickness 0.15)) (justify left mirror))
   )
